File: hardware/netlist/single_channel.kicad_sch (KiCad schematic)
At the start: 23 parts, among them J1 BNC (insect electrode), J2 Lemo/ODU 8-pin to motherboard, K1 latching reed relay (Ri sw), U3 ADA4940-1 FDA (gain + diff dr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, U4 latching-relay driver (H-brid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

Commit message: hardware: PCB layout groundwork + hand-off (footprints, placed board, spec, DRU)
Assign KiCad footprints (netlist + schematic Footprint properties; 3 PLACEHOLDERs).
Generate a pre-placed single_channel.kicad_pcb via the pcbnew API (electrometer-aware
placement, 60x40mm, 4 layers; kicad-cli DRC: 0 structural errors, 40 placement-
refinement items). Add pcb-layout.md (stackup, guard rings, Cin<=1pF rules, net
classes, grounding) and single_channel.kicad_dru (custom rules, parse-validated).

Co-Authored-By: Claude Opus 4.8 (1M context) <noreply@anthropic.com>
Parts:
- A1, A2: footprint (none) -> Package_SO:SOIC-8_3.9x4.9mm_P1.27mm
- C1, C2, C3, C4, C5, C6, CV: footprint (none) -> Capacitor_SMD:C_0603_1608Metric
- J1: footprint (none) -> Connector_Coaxial:BNC_Amphenol_031-5539_Vertical
- J2: footprint (none) -> Connector_PinHeader_2.54mm:PinHeader_1x08_P2.54mm_Vertical
- K1: footprint (none) -> Relay_THT:Relay_1-Form-A_Schrack-RYII_RM5mm
- RF1, RF2, RG1, RG2, RO1, RO2, RV1, RV2: footprint (none) -> Resistor_SMD:R_0603_1608Metric
- RI: footprint (none) -> Resistor_SMD:R_1206_3216Metric
- U3: footprint (none) -> Package_DFN_QFN:HVQFN-16-1EP_3x3mm_P0.5mm_EP1.5x1.5mm
- U4: footprint (none) -> Package_TO_SOT_SMD:SOT-23-6
